File: Isolated_DCDC_Converter.kicad_pcb (KiCad board)
At the start: 2 copper layers, 80 x 25 mm, 23 parts, among them U1 LMR51635YDDCR

Commit message: Added Copper Pours
Parts:
- moved C7 7.00 mm to (179.8, 57.3)
Routing:
- net ISO GND: track 1.60 -> 8.29 mm, vias 11 -> 5
- added copper zone on F.Cu, net BAT GND
- added copper zone on F.Cu, net Net-(MD1-+VIN)
Changed lines of the file:
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@@
 	(footprint "Capacitor_SMD:C_0603_1608Metric_Pad1.08x0.95mm_HandSolder"
 		(layer "F.Cu")
-		(at 179.85 50.3)
+		(at 179.85 57.3)
 		(descr "Capacitor SMD 0603 (1608 Metric), square (rectangular) end terminal, IPC-7351 nominal with elongated pad for handsoldering. (Body size source: IPC-SM-782 page 76, https://www.pcb-3d.com/wordpress/wp-content/uploads/ipc-sm-782a_amendment_1_and_2.pdf)")
 		(tags "capacitor handsolder")
 		(property "Reference" "C7"
-			(at 0.75 -1.45 0)
+			(at -0.7 1.8 0)
 			(layer "F.SilkS")
 			(effects
@@
 	)
 	(segment
+		(start 175.325 41.625)
+		(end 175.325 43.145)
+		(width 0.5)
+		(layer "F.Cu")
+		(net "ISO GND")
+	)
+	(segment
+		(start 180.712501 57.3)
+		(end 182.212501 57.3)
+		(width 0.5)
+		(layer "F.Cu")
+		(net "ISO GND")
+	)
+	(segment
 		(start 172.069992 47.674991)
 		(end 171.5825 47.187498)
@@
 	)
 	(segment
+		(start 175.325 41.625)
+		(end 177.49 41.624999)
+		(width 0.5)
+		(layer "F.Cu")
+		(net "ISO GND")
+	)
+	(segment
+		(start 178.95 43.474998)
+		(end 178.95 44.974998)
+		(width 0.5)
+		(layer "F.Cu")
+		(net "ISO GND")
+	)
+	(segment
 		(start 171.5825 47.187498)
 		(end 171.15 47.187498)
 		(width 0.5)
 		(layer "F.Cu")
-		(net "ISO GND")
-	)
-	(via
-		(at 157.3 49.95)
-		(size 0.8)
-		(drill 0.3)
-		(layers "F.Cu" "B.Cu")
-		(free yes)
-		(net "ISO GND")
-	)
-	(via
-		(at 166.3 50.9)
-		(size 0.8)
-		(drill 0.3)
-		(layers "F.Cu" "B.Cu")
-		(free yes)
 		(net "ISO GND")
 	)
@@
 	)
 	(via
-		(at 161.25 48.9)
+		(at 175.325 41.625)
 		(size 0.8)
 		(drill 0.3)
 		(layers "F.Cu" "B.Cu")
-		(free yes)
+		(teardrops
+			(best_length_ratio 0.5)
+			(max_length 1)
+			(best_width_ratio 1)
+			(max_width 2)
+			(curved_edges no)
+			(filter_ratio 0.9)
+			(enabled yes)
+			(allow_two_segments yes)
+			(prefer_zone_connections yes)
+		)
 		(net "ISO GND")
 	)
@@
 	)
 	(via
-		(at 166 49.3)
+		(at 178.95 43.474998)
 		(size 0.8)
 		(drill 0.3)
 		(layers "F.Cu" "B.Cu")
-		(free yes)
+		(teardrops
+			(best_length_ratio 0.5)
+			(max_length 1)
+			(best_width_ratio 1)
+			(max_width 2)
+			(curved_edges no)
+			(filter_ratio 0.9)
+			(enabled yes)
+			(allow_two_segments yes)
+			(prefer_zone_connections yes)
+		)
 		(net "ISO GND")
 	)
 	(via
-		(at 150.85 58.75)
+		(at 182.212501 57.3)
 		(size 0.8)
 		(drill 0.3)
 		(layers "F.Cu" "B.Cu")
-		(free yes)
-		(net "ISO GND")
-	)
-	(via
-		(at 161.25 50.75)
-		(size 0.8)
-		(drill 0.3)
-		(layers "F.Cu" "B.Cu")
-		(free yes)
-		(net "ISO GND")
-	)
-	(via
-		(at 158.2 49.8)
-		(size 0.8)
-		(drill 0.3)
-		(layers "F.Cu" "B.Cu")
-		(free yes)
-		(net "ISO GND")
-	)
-	(via
-		(at 167.55 52.15)
-		(size 0.8)
-		(drill 0.3)
-		(layers "F.Cu" "B.Cu")
-		(free yes)
-		(net "ISO GND")
-	)
-	(via
-		(at 167.85 51.45)
-		(size 0.8)
-		(drill 0.3)
-		(layers "F.Cu" "B.Cu")
-		(free yes)
+		(teardrops
+			(best_length_ratio 0.5)
+			(max_length 1)
+			(best_width_ratio 1)
+			(max_width 2)
+			(curved_edges no)
+			(filter_ratio 0.9)
+			(enabled yes)
+			(allow_two_segments yes)
+			(prefer_zone_connections yes)
+		)
 		(net "ISO GND")
 	)
@@
 		(layer "F.Cu")
 		(net "Net-(U1-CB)")
+	)
+	(zone
+		(net "Net-(MD1-+VIN)")
+		(layer "F.Cu")
+		(hatch edge 0.5)
+		(priority 6)
+		(connect_pads
+			(clearance 0.25)
+		)
+		(min_thickness 0.1)
+		(fill yes
+			(thermal_gap 0.2)
+			(thermal_bridge_width 0.75)
+			(smoothing fillet)
+			(radius 1)
+			(island_removal_mode 0)
+		)
+		(polygon
+			(pts
+				(xy 118.25 65.5) (xy 118.25 56.3) (xy 129.4 56.3) (xy 129.4 40.4) (xy 124.05 40.4) (xy 124.05 51.95)
+				(xy 112.95 51.95) (xy 112.95 65.5)
+			)
+		)
+	)
+	(zone
+		(net "ISO GND")
+		(layer "F.Cu")
+		(hatch none 0.1)
+		(priority 30005)
+		(attr
+			(teardrop
+				(type padvia)
+			)
+		)
+		(connect_pads yes
+			(clearance 0)
+		)
+		(min_thickness 0.0254)
+		(fill yes
+			(island_removal_mode 1)
+		)
+		(polygon
+			(pts
+				(xy 175.075 42.421578) (xy 175.575 42.421578) (xy 175.721578 41.67721) (xy 175.325 41.620578) (xy 174.928422 41.67721)
+			)
+		)
 	)
 	(zone
@@
 		(layer "F.Cu")
 		(hatch none 0.1)
-		(priority 30007)
+		(priority 30011)
 		(attr
 			(teardrop
@@
 		(layer "F.Cu")
 		(hatch none 0.1)
-		(priority 30005)
+		(priority 30009)
 		(attr
 			(teardrop
@@
 	)
 	(zone
+		(net "ISO GND")
+		(layer "F.Cu")
+		(hatch none 0.1)
+		(priority 30008)
+		(attr
+			(teardrop
+				(type padvia)
+			)
+		)
+		(connect_pads yes
+			(clearance 0)
+		)
+		(min_thickness 0.0254)
+		(fill yes
+			(island_removal_mode 1)
+		)
+		(polygon
+			(pts
+				(xy 176.121578 41.874999) (xy 176.121577 41.375) (xy 175.37721 41.228422) (xy 175.320578 41.625)
+				(xy 175.37721 42.021578)
+			)
+		)
+	)
+	(zone
 		(net "Net-(U1-SW)")
 		(layer "F.Cu")
@@
 	)
 	(zone
+		(net "ISO GND")
+		(layer "F.Cu")
+		(hatch none 0.1)
+		(priority 30006)
+		(attr
+			(teardrop
+				(type padvia)
+			)
+		)
+		(connect_pads yes
+			(clearance 0)
+		)
+		(min_thickness 0.0254)
+		(fill yes
+			(island_removal_mode 1)
+		)
+		(polygon
+			(pts
+				(xy 178.7 44.271576) (xy 179.2 44.271576) (xy 179.346578 43.527208) (xy 178.95 43.470576) (xy 178.553422 43.527208)
+			)
+		)
+	)
+	(zone
+		(net "ISO GND")
+		(layer "F.Cu")
+		(hatch none 0.1)
+		(priority 30007)
+		(attr
+			(teardrop
+				(type padvia)
+			)
+		)
+		(connect_pads yes
+			(clearance 0)
+		)
+		(min_thickness 0.0254)
+		(fill yes
+			(island_removal_mode 1)
+		)
+		(polygon
+			(pts
+				(xy 181.415923 57.05) (xy 181.415923 57.55) (xy 182.160291 57.696578) (xy 182.216923 57.3) (xy 182.160291 56.903422)
+			)
+		)
+	)
+	(zone
 		(net "Net-(U1-SW)")
 		(layer "F.Cu")
@@
 		(layer "F.Cu")
 		(hatch none 0.1)
-		(priority 30006)
+		(priority 30010)
 		(attr
 			(teardrop
@@
 				(xy 172.196168 44.757627) (xy 172.118535 44.738551) (xy 172.069992 44.725007) (xy 171.893215 44.79823)
 				(xy 171.808368 44.883079)
+			)
+		)
+	)
+	(zone
+		(net "BAT GND")
+		(layer "F.Cu")
+		(hatch edge 0.5)
+		(priority 5)
+		(connect_pads
+			(clearance 0.25)
+		)
+		(min_thickness 0.1)
+		(fill yes
+			(thermal_gap 0.2)
+			(thermal_bridge_width 0.75)
+			(smoothing fillet)
+			(radius 1)
+			(island_removal_mode 0)
+		)
+		(polygon
+			(pts
+				(xy 129.4 57.65) (xy 129.4 65.5) (xy 118.95 65.5) (xy 118.95 57.65)
 			)
 		)
@@
 		(polygon
 			(pts
-				(xy 128.25 38.75) (xy 128.25 65.5) (xy 104 65.5) (xy 104 38.75)
-			)
-		)
+				(xy 129.4 38.75) (xy 129.4 65.5) (xy 104 65.5) (xy 104 38.75)
+			)
+		)
